File: pcb/more-organic/more-organic.sch (KiCad schematic (older format))
At the start: 67 parts, among them SW1 SW_Push, SW10 SW_Push, SW11 SW_Push, SW12 SW_Push, SW13 SW_Push, SW14 SW_Push, SW15 SW_Push, SW16 SW_Push, SW17 SW_Push, SW18 SW_Push, SW19 SW_Push, SW2 SW_Push, SW20 SW_Push, SW21 SW_Push, SW22 SW_Push, SW23 SW_Push, SW24 SW_Push, SW25 SW_Push, SW26 SW_Push, SW27 SW_Push, SW28 SW_Push, SW29 SW_Push, SW3 SW_Push, SW30 SW_Push, SW31 MX, SW4 SW_Push, SW5 SW_Push, SW6 SW_Push, SW7 SW_Push, SW8 SW_Push, SW9 SW_Push, U1 ProMicro, U2 TRRS

Commit message: Add readme, images
Parts:
- SW1, SW10, SW11, SW12, SW13, SW14, SW15, SW16, SW17, SW18, SW19, SW2, SW20, SW21, SW22, SW23, SW24, SW25, SW26, SW27, SW28, SW29, SW3, SW30, SW4, SW5, SW6, SW7, SW8, SW9: footprint keyswitches:SW_MX_reversible -> keyswitches:Kailh_socket_MX_optional_reversible_alt
Changed lines of the file:
@@
 F 0 "SW1" H 5700 1300 50  0000 C CNN
 F 1 "SW_Push" H 5700 1200 50  0000 C CNN
-F 2 "keyswitches:SW_MX_reversible" H 5700 1200 50  0001 C CNN
+F 2 "keyswitches:Kailh_socket_MX_optional_reversible_alt" H 5700 1200 50  0001 C CNN
 F 3 "~" H 5700 1200 50  0001 C CNN
 	1    5700 1000
@@
 F 0 "SW2" H 6700 1300 50  0000 C CNN
 F 1 "SW_Push" H 6700 1200 50  0000 C CNN
-F 2 "keyswitches:SW_MX_reversible" H 6700 1200 50  0001 C CNN
+F 2 "keyswitches:Kailh_socket_MX_optional_reversible_alt" H 6700 1200 50  0001 C CNN
 F 3 "~" H 6700 1200 50  0001 C CNN
 	1    6700 1000
@@
 F 0 "SW3" H 7700 1300 50  0000 C CNN
 F 1 "SW_Push" H 7700 1200 50  0000 C CNN
-F 2 "keyswitches:SW_MX_reversible" H 7700 1200 50  0001 C CNN
+F 2 "keyswitches:Kailh_socket_MX_optional_reversible_alt" H 7700 1200 50  0001 C CNN
 F 3 "~" H 7700 1200 50  0001 C CNN
 	1    7700 1000
@@
 F 0 "SW4" H 8700 1300 50  0000 C CNN
 F 1 "SW_Push" H 8700 1200 50  0000 C CNN
-F 2 "keyswitches:SW_MX_reversible" H 8700 1200 50  0001 C CNN
+F 2 "keyswitches:Kailh_socket_MX_optional_reversible_alt" H 8700 1200 50  0001 C CNN
 F 3 "~" H 8700 1200 50  0001 C CNN
 	1    8700 1000
@@
 F 0 "SW5" H 9700 1300 50  0000 C CNN
 F 1 "SW_Push" H 9700 1200 50  0000 C CNN
-F 2 "keyswitches:SW_MX_reversible" H 9700 1200 50  0001 C CNN
+F 2 "keyswitches:Kailh_socket_MX_optional_reversible_alt" H 9700 1200 50  0001 C CNN
 F 3 "~" H 9700 1200 50  0001 C CNN
 	1    9700 1000
@@
 F 0 "SW6" H 10700 1300 50  0000 C CNN
 F 1 "SW_Push" H 10700 1200 50  0000 C CNN
-F 2 "keyswitches:SW_MX_reversible" H 10700 1200 50  0001 C CNN
+F 2 "keyswitches:Kailh_socket_MX_optional_reversible_alt" H 10700 1200 50  0001 C CNN
 F 3 "~" H 10700 1200 50  0001 C CNN
 	1    10700 1000
@@
 F 0 "SW7" H 5700 2300 50  0000 C CNN
 F 1 "SW_Push" H 5700 2200 50  0000 C CNN
-F 2 "keyswitches:SW_MX_reversible" H 5700 2200 50  0001 C CNN
+F 2 "keyswitches:Kailh_socket_MX_optional_reversible_alt" H 5700 2200 50  0001 C CNN
 F 3 "~" H 5700 2200 50  0001 C CNN
 	1    5700 2000
@@
 F 0 "SW8" H 6700 2300 50  0000 C CNN
 F 1 "SW_Push" H 6700 2200 50  0000 C CNN
-F 2 "keyswitches:SW_MX_reversible" H 6700 2200 50  0001 C CNN
+F 2 "keyswitches:Kailh_socket_MX_optional_reversible_alt" H 6700 2200 50  0001 C CNN
 F 3 "~" H 6700 2200 50  0001 C CNN
 	1    6700 2000
@@
 F 0 "SW9" H 7700 2300 50  0000 C CNN
 F 1 "SW_Push" H 7700 2200 50  0000 C CNN
-F 2 "keyswitches:SW_MX_reversible" H 7700 2200 50  0001 C CNN
+F 2 "keyswitches:Kailh_socket_MX_optional_reversible_alt" H 7700 2200 50  0001 C CNN
 F 3 "~" H 7700 2200 50  0001 C CNN
 	1    7700 2000
@@
 F 0 "SW10" H 8700 2300 50  0000 C CNN
 F 1 "SW_Push" H 8700 2200 50  0000 C CNN
-F 2 "keyswitches:SW_MX_reversible" H 8700 2200 50  0001 C CNN
+F 2 "keyswitches:Kailh_socket_MX_optional_reversible_alt" H 8700 2200 50  0001 C CNN
 F 3 "~" H 8700 2200 50  0001 C CNN
 	1    8700 2000
@@
 F 0 "SW11" H 9700 2300 50  0000 C CNN
 F 1 "SW_Push" H 9700 2200 50  0000 C CNN
-F 2 "keyswitches:SW_MX_reversible" H 9700 2200 50  0001 C CNN
+F 2 "keyswitches:Kailh_socket_MX_optional_reversible_alt" H 9700 2200 50  0001 C CNN
 F 3 "~" H 9700 2200 50  0001 C CNN
 	1    9700 2000
@@
 F 0 "SW12" H 10700 2300 50  0000 C CNN
 F 1 "SW_Push" H 10700 2200 50  0000 C CNN
-F 2 "keyswitches:SW_MX_reversible" H 10700 2200 50  0001 C CNN
+F 2 "keyswitches:Kailh_socket_MX_optional_reversible_alt" H 10700 2200 50  0001 C CNN
 F 3 "~" H 10700 2200 50  0001 C CNN
 	1    10700 2000
@@
 F 0 "SW13" H 5700 3300 50  0000 C CNN
 F 1 "SW_Push" H 5700 3200 50  0000 C CNN
-F 2 "keyswitches:SW_MX_reversible" H 5700 3200 50  0001 C CNN
+F 2 "keyswitches:Kailh_socket_MX_optional_reversible_alt" H 5700 3200 50  0001 C CNN
 F 3 "~" H 5700 3200 50  0001 C CNN
 	1    5700 3000
@@
 F 0 "SW14" H 6700 3300 50  0000 C CNN
 F 1 "SW_Push" H 6700 3200 50  0000 C CNN
-F 2 "keyswitches:SW_MX_reversible" H 6700 3200 50  0001 C CNN
+F 2 "keyswitches:Kailh_socket_MX_optional_reversible_alt" H 6700 3200 50  0001 C CNN
 F 3 "~" H 6700 3200 50  0001 C CNN
 	1    6700 3000
@@
 F 0 "SW15" H 7700 3300 50  0000 C CNN
 F 1 "SW_Push" H 7700 3200 50  0000 C CNN
-F 2 "keyswitches:SW_MX_reversible" H 7700 3200 50  0001 C CNN
+F 2 "keyswitches:Kailh_socket_MX_optional_reversible_alt" H 7700 3200 50  0001 C CNN
 F 3 "~" H 7700 3200 50  0001 C CNN
 	1    7700 3000
@@
 F 0 "SW16" H 8700 3300 50  0000 C CNN
 F 1 "SW_Push" H 8700 3200 50  0000 C CNN
-F 2 "keyswitches:SW_MX_reversible" H 8700 3200 50  0001 C CNN
+F 2 "keyswitches:Kailh_socket_MX_optional_reversible_alt" H 8700 3200 50  0001 C CNN
 F 3 "~" H 8700 3200 50  0001 C CNN
 	1    8700 3000
@@
 F 0 "SW17" H 9700 3300 50  0000 C CNN
 F 1 "SW_Push" H 9700 3200 50  0000 C CNN
-F 2 "keyswitches:SW_MX_reversible" H 9700 3200 50  0001 C CNN
+F 2 "keyswitches:Kailh_socket_MX_optional_reversible_alt" H 9700 3200 50  0001 C CNN
 F 3 "~" H 9700 3200 50  0001 C CNN
 	1    9700 3000
@@
 F 0 "SW18" H 10700 3300 50  0000 C CNN
 F 1 "SW_Push" H 10700 3200 50  0000 C CNN
-F 2 "keyswitches:SW_MX_reversible" H 10700 3200 50  0001 C CNN
+F 2 "keyswitches:Kailh_socket_MX_optional_reversible_alt" H 10700 3200 50  0001 C CNN
 F 3 "~" H 10700 3200 50  0001 C CNN
 	1    10700 3000
@@
 F 0 "SW19" H 5700 4300 50  0000 C CNN
 F 1 "SW_Push" H 5700 4200 50  0000 C CNN
-F 2 "keyswitches:SW_MX_reversible" H 5700 4200 50  0001 C CNN
+F 2 "keyswitches:Kailh_socket_MX_optional_reversible_alt" H 5700 4200 50  0001 C CNN
 F 3 "~" H 5700 4200 50  0001 C CNN
 	1    5700 4000
@@
 F 0 "SW20" H 6700 4300 50  0000 C CNN
 F 1 "SW_Push" H 6700 4200 50  0000 C CNN
-F 2 "keyswitches:SW_MX_reversible" H 6700 4200 50  0001 C CNN
+F 2 "keyswitches:Kailh_socket_MX_optional_reversible_alt" H 6700 4200 50  0001 C CNN
 F 3 "~" H 6700 4200 50  0001 C CNN
 	1    6700 4000
@@
 F 0 "SW21" H 7700 4300 50  0000 C CNN
 F 1 "SW_Push" H 7700 4200 50  0000 C CNN
-F 2 "keyswitches:SW_MX_reversible" H 7700 4200 50  0001 C CNN
+F 2 "keyswitches:Kailh_socket_MX_optional_reversible_alt" H 7700 4200 50  0001 C CNN
 F 3 "~" H 7700 4200 50  0001 C CNN
 	1    7700 4000
@@
 F 0 "SW22" H 8700 4300 50  0000 C CNN
 F 1 "SW_Push" H 8700 4200 50  0000 C CNN
-F 2 "keyswitches:SW_MX_reversible" H 8700 4200 50  0001 C CNN
+F 2 "keyswitches:Kailh_socket_MX_optional_reversible_alt" H 8700 4200 50  0001 C CNN
 F 3 "~" H 8700 4200 50  0001 C CNN
 	1    8700 4000
@@
 F 0 "SW23" H 9700 4300 50  0000 C CNN
 F 1 "SW_Push" H 9700 4200 50  0000 C CNN
-F 2 "keyswitches:SW_MX_reversible" H 9700 4200 50  0001 C CNN
+F 2 "keyswitches:Kailh_socket_MX_optional_reversible_alt" H 9700 4200 50  0001 C CNN
 F 3 "~" H 9700 4200 50  0001 C CNN
 	1    9700 4000
@@
 F 0 "SW24" H 10700 4300 50  0000 C CNN
 F 1 "SW_Push" H 10700 4200 50  0000 C CNN
-F 2 "keyswitches:SW_MX_reversible" H 10700 4200 50  0001 C CNN
+F 2 "keyswitches:Kailh_socket_MX_optional_reversible_alt" H 10700 4200 50  0001 C CNN
 F 3 "~" H 10700 4200 50  0001 C CNN
 	1    10700 4000
@@
 F 0 "SW25" H 5700 5300 50  0000 C CNN
 F 1 "SW_Push" H 5700 5200 50  0000 C CNN
-F 2 "keyswitches:SW_MX_reversible" H 5700 5200 50  0001 C CNN
+F 2 "keyswitches:Kailh_socket_MX_optional_reversible_alt" H 5700 5200 50  0001 C CNN
 F 3 "~" H 5700 5200 50  0001 C CNN
 	1    5700 5000
@@
 F 0 "SW26" H 6700 5300 50  0000 C CNN
 F 1 "SW_Push" H 6700 5200 50  0000 C CNN
-F 2 "keyswitches:SW_MX_reversible" H 6700 5200 50  0001 C CNN
+F 2 "keyswitches:Kailh_socket_MX_optional_reversible_alt" H 6700 5200 50  0001 C CNN
 F 3 "~" H 6700 5200 50  0001 C CNN
 	1    6700 5000
@@
 F 0 "SW27" H 7700 5300 50  0000 C CNN
 F 1 "SW_Push" H 7700 5200 50  0000 C CNN
-F 2 "keyswitches:SW_MX_reversible" H 7700 5200 50  0001 C CNN
+F 2 "keyswitches:Kailh_socket_MX_optional_reversible_alt" H 7700 5200 50  0001 C CNN
 F 3 "~" H 7700 5200 50  0001 C CNN
 	1    7700 5000
@@
 F 0 "SW28" H 8700 5300 50  0000 C CNN
 F 1 "SW_Push" H 8700 5200 50  0000 C CNN
-F 2 "keyswitches:SW_MX_reversible" H 8700 5200 50  0001 C CNN
+F 2 "keyswitches:Kailh_socket_MX_optional_reversible_alt" H 8700 5200 50  0001 C CNN
 F 3 "~" H 8700 5200 50  0001 C CNN
 	1    8700 5000
@@
 F 0 "SW29" H 9700 5300 50  0000 C CNN
 F 1 "SW_Push" H 9700 5200 50  0000 C CNN
-F 2 "keyswitches:SW_MX_reversible" H 9700 5200 50  0001 C CNN
+F 2 "keyswitches:Kailh_socket_MX_optional_reversible_alt" H 9700 5200 50  0001 C CNN
 F 3 "~" H 9700 5200 50  0001 C CNN
 	1    9700 5000
@@
 F 0 "SW30" H 10700 5300 50  0000 C CNN
 F 1 "SW_Push" H 10700 5200 50  0000 C CNN
-F 2 "keyswitches:SW_MX_reversible" H 10700 5200 50  0001 C CNN
+F 2 "keyswitches:Kailh_socket_MX_optional_reversible_alt" H 10700 5200 50  0001 C CNN
 F 3 "~" H 10700 5200 50  0001 C CNN
 	1    10700 5000

Commit message: Update pcb with recent placement, remove 3 not used switches
Parts:
- removed D28, D29, D30: D, keebio-footprints:Diode-dual, symbol Device:D
- removed SW28, SW29, SW30: SW_Push, keyswitches:Kailh_socket_MX_optional_reversible_alt, symbol Switch:SW_Push
- renumbered SW31 to SW_RESET1
Changed lines of the file:
@@
 $EndComp
 $Comp
-L Switch:SW_Push SW31
+L Switch:SW_Push SW_RESET1
 U 1 1 5F33BD98
 P 3850 6200
-F 0 "SW31" H 3850 6400 50  0000 C CNN
+F 0 "SW_RESET1" H 3850 6400 50  0000 C CNN
 F 1 "MX" H 3850 5900 60  0001 C CNN
 F 2 "Button_Switch_THT:SW_PUSH_6mm_H7.3mm" H 3850 6200 60  0001 C CNN
@@
 Wire Wire Line
 	7900 5300 7900 5500
-$Comp
-L Switch:SW_Push SW28
-U 1 1 5F33BF9C
-P 8700 5000
-F 0 "SW28" H 8700 5300 50  0000 C CNN
-F 1 "SW_Push" H 8700 5200 50  0000 C CNN
-F 2 "keyswitches:Kailh_socket_MX_optional_reversible_alt" H 8700 5200 50  0001 C CNN
-F 3 "~" H 8700 5200 50  0001 C CNN
-	1    8700 5000
-	1    0    0    -1
-$EndComp
-$Comp
-L Device:D D28
-U 1 1 5F33BFA2
-P 8900 5150
-F 0 "D28" V 8950 5250 50  0000 L CNN
-F 1 "D" V 8900 5250 50  0000 L CNN
-F 2 "keebio-footprints:Diode-dual" H 8900 5150 50  0001 C CNN
-F 3 "~" H 8900 5150 50  0001 C CNN
-	1    8900 5150
-	0    1    -1   0
-$EndComp
-Wire Wire Line
-	8500 5000 8400 5000
-Wire Wire Line
-	8900 5300 8900 5500
-$Comp
-L Switch:SW_Push SW29
-U 1 1 5F33BFAA
-P 9700 5000
-F 0 "SW29" H 9700 5300 50  0000 C CNN
-F 1 "SW_Push" H 9700 5200 50  0000 C CNN
-F 2 "keyswitches:Kailh_socket_MX_optional_reversible_alt" H 9700 5200 50  0001 C CNN
-F 3 "~" H 9700 5200 50  0001 C CNN
-	1    9700 5000
-	1    0    0    -1
-$EndComp
-$Comp
-L Device:D D29
-U 1 1 5F33BFB0
-P 9900 5150
-F 0 "D29" V 9950 5250 50  0000 L CNN
-F 1 "D" V 9900 5250 50  0000 L CNN
-F 2 "keebio-footprints:Diode-dual" H 9900 5150 50  0001 C CNN
-F 3 "~" H 9900 5150 50  0001 C CNN
-	1    9900 5150
-	0    1    -1   0
-$EndComp
-Wire Wire Line
-	9500 5000 9400 5000
-Wire Wire Line
-	9900 5300 9900 5500
-$Comp
-L Switch:SW_Push SW30
-U 1 1 5F33BFB8
-P 10700 5000
-F 0 "SW30" H 10700 5300 50  0000 C CNN
-F 1 "SW_Push" H 10700 5200 50  0000 C CNN
-F 2 "keyswitches:Kailh_socket_MX_optional_reversible_alt" H 10700 5200 50  0001 C CNN
-F 3 "~" H 10700 5200 50  0001 C CNN
-	1    10700 5000
-	1    0    0    -1
-$EndComp
-$Comp
-L Device:D D30
-U 1 1 5F33BFBE
-P 10900 5150
-F 0 "D30" V 10950 5250 50  0000 L CNN
-F 1 "D" V 10900 5250 50  0000 L CNN
-F 2 "keebio-footprints:Diode-dual" H 10900 5150 50  0001 C CNN
-F 3 "~" H 10900 5150 50  0001 C CNN
-	1    10900 5150
-	0    1    -1   0
-$EndComp
-Wire Wire Line
-	10500 5000 10400 5000
-Wire Wire Line
-	10900 5300 10900 5500
 Wire Wire Line
 	10900 2500 9900 2500
@@
 Wire Wire Line
 	9900 4500 8900 4500
-Wire Wire Line
-	10900 5500 9900 5500
 Connection ~ 5900 5500
 Wire Wire Line
@@
 Wire Wire Line
 	6900 5500 5900 5500
-Connection ~ 7900 5500
 Wire Wire Line
 	7900 5500 6900 5500
-Connection ~ 8900 5500
-Wire Wire Line
-	8900 5500 7900 5500
-Connection ~ 9900 5500
-Wire Wire Line
-	9900 5500 8900 5500
 Wire Wire Line
 	5400 5000 5400 4000
@@
 Wire Wire Line
 	8400 3000 8400 4000
-Connection ~ 8400 4000
-Wire Wire Line
-	8400 4000 8400 5000
-Wire Wire Line
-	9400 5000 9400 4000
 Connection ~ 9400 2000
 Wire Wire Line
@@
 Wire Wire Line
 	9400 3000 9400 2000
-Connection ~ 9400 4000
 Wire Wire Line
 	9400 4000 9400 3000
@@
 Wire Wire Line
 	10400 3000 10400 4000
-Connection ~ 10400 4000
-Wire Wire Line
-	10400 4000 10400 5000
 Wire Wire Line
 	10400 1000 10200 1000
