File: pcb/more-organic/more-organic.kicad_pcb (KiCad board)
At the start: 2 copper layers, 67 parts, among them SW1 SW_Push, SW10 SW_Push, SW11 SW_Push, SW12 SW_Push, SW13 SW_Push, SW14 SW_Push, SW15 SW_Push, SW16 SW_Push, SW17 SW_Push, SW18 SW_Push, SW19 SW_Push, SW2 SW_Push, SW20 SW_Push, SW21 SW_Push, SW22 SW_Push, SW23 SW_Push, SW24 SW_Push, SW25 SW_Push, SW26 SW_Push, SW27 SW_Push, SW28 SW_Push, SW29 SW_Push, SW3 SW_Push, SW30 SW_Push, SW31 MX, SW4 SW_Push, SW5 SW_Push, SW6 SW_Push, SW7 SW_Push, SW8 SW_Push, SW9 SW_Push, U1 ProMicro, U2 TRRS

Commit message: Add readme, images
Parts:
- SW1, SW10, SW11, SW12, SW13, SW14, SW15, SW16, SW17, SW18, SW19, SW2, SW20, SW21, SW22, SW23, SW24, SW25, SW26, SW27, SW28, SW29, SW3, SW30, SW4, SW5, SW6, SW7, SW8, SW9: footprint keyswitches:SW_MX_reversible -> keyswitches:Kailh_socket_MX_optional_reversible_alt
- moved JP2 219.2 mm to (75.1, 74.3), turned to 90 degrees
- moved JP1 213.2 mm to (75.1, 78.6), turned to 90 degrees
- moved R1 211.4 mm to (74.2, 67.5), turned to 90 degrees
- moved R2 203.0 mm to (74.9, 86.0), turned to 90 degrees
- moved U2 60.1 mm to (104.2, 54.0)
- moved SW27 13.6 mm to (151.1, 142.6), turned to 330 degrees
- moved D19 12.8 mm to (119.0, 110.1), turned to 180 degrees
- moved D8 12.8 mm to (138.1, 69.6), turned to 180 degrees
- moved D10 12.8 mm to (176.2, 69.6), turned to 180 degrees
- moved D13 12.8 mm to (119.0, 91.0), turned to 180 degrees
- moved D14 12.8 mm to (138.1, 88.6), turned to 180 degrees
- moved D20 12.8 mm to (138.1, 107.7), turned to 180 degrees
- moved D7 12.8 mm to (119.0, 72.0), turned to 180 degrees
- moved D1 12.8 mm to (119.0, 52.9), turned to 180 degrees
- moved D2 12.8 mm to (138.1, 50.5), turned to 180 degrees
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Routing:
- net /col5: track 0.00 -> 277.1 mm, vias 0 -> 5
- net /col4: track 0.00 -> 255.4 mm, vias 0 -> 5
- net /col3: track 0.00 -> 240.7 mm, vias 0 -> 5
- net /col2: track 0.00 -> 216.2 mm, vias 0 -> 5
- net /col1: track 0.00 -> 193.5 mm, vias 0 -> 5
- net /col0: track 0.00 -> 168.8 mm, vias 0 -> 5
- net /row3: track 0.00 -> 121.9 mm
- net /row2: track 0.00 -> 118.5 mm
- net /row0: track 0.00 -> 117.9 mm
- net /row1: track 0.00 -> 104.4 mm
- net /row4: track 0.00 -> 88.4 mm
- net Net-(D1-Pad2): track 0.00 -> 24.7 mm
- net Net-(D24-Pad2): track 0.00 -> 7.50 mm, vias 0 -> 1

Commit message: Update pcb with recent placement, remove 3 not used switches
Parts:
- moved U2 153.2 mm to (-40.0, 2.00)
- moved SW10 136.6 mm to (57.1, 11.1)
- moved SW16 136.6 mm to (57.1, 30.1)
- moved SW22 136.6 mm to (57.1, 49.1)
- moved SW4 136.6 mm to (57.1, -8.00)
- moved SW15 136.3 mm to (38.1, 26.1)
- moved SW21 136.3 mm to (38.1, 45.1)
- moved SW3 136.3 mm to (38.1, -12.0)
- moved SW9 136.3 mm to (38.1, 7.05)
- moved D27 134.2 mm to (27.8, 93.6)
- moved SW14 132.9 mm to (19.1, 38.1)
- moved SW2 132.9 mm to (19.1, 0.00)
- moved SW20 132.9 mm to (19.1, 57.1)
- moved SW8 132.9 mm to (19.1, 19.1)
- moved SW1 131.7 mm to (0.00, 5.00)
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- renumbered SW31 to SW_RESET1
Routing:
- net /col4: track 255.4 -> 13.7 mm, vias 5 -> 1
- net /col3: track 240.7 -> 16.1 mm, vias 5 -> 1
- net /col2: track 216.2 -> 0.00 mm, vias 5 -> 0
- net /col1: track 193.5 -> 0.00 mm, vias 5 -> 0
- net /col0: track 168.8 -> 0.00 mm, vias 5 -> 0
- net /row3: track 121.9 -> 0.00 mm
- net /row2: track 118.5 -> 0.00 mm
- net /row0: track 117.9 -> 0.00 mm
- net /col5: track 277.1 -> 166.0 mm, vias 5 -> 1
- net /row1: track 104.4 -> 0.00 mm
- net /row4: track 88.4 -> 0.00 mm
- net Net-(D1-Pad2): track 24.7 -> 0.00 mm
- net /xtradata: track 0.00 -> 13.7 mm
- net VCC: track 0.00 -> 12.5 mm
- net /sda: track 0.00 -> 11.6 mm
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Other:
- board outline added: 156.4 x 122.7 mm

Commit message: Redesigning makefile, design and pcb data flow
Parts:
- removed D28, D29, D30: D, keebio-footprints:Diode-dual
- removed SW28, SW29, SW30: SW_Push, keyswitches:Kailh_socket_MX_optional_reversible_alt
- added REF**: MountingHole_2.2mm_M2_Pad_Via, MountingHole_2.2mm_M2_Pad_Via, F.Cu at (-20.0, 30.0)
- added REF**: MountingHole_2.2mm_M2_Pad_Via, MountingHole_2.2mm_M2_Pad_Via, F.Cu at (63.7, 61.7)
- added REF**: MountingHole_2.2mm_M2_Pad_Via, MountingHole_2.2mm_M2_Pad_Via, F.Cu at (12.0, 69.2)
- added REF**: MountingHole_2.2mm_M2_Pad_Via, MountingHole_2.2mm_M2_Pad_Via, F.Cu at (69.7, 5.47)
- added REF**: MountingHole_2.2mm_M2_Pad_Via, MountingHole_2.2mm_M2_Pad_Via, F.Cu at (25.6, -12.5)
Routing:
- net /col3: track 16.1 -> 0.00 mm, vias 1 -> 0
- net /col4: track 13.7 -> 0.00 mm, vias 1 -> 0
- net /col5: track 166.0 -> 152.3 mm, vias 1 -> 0
